File: STM32Scope.sch (KiCad schematic (older format))
At the start: 11 parts, among them J101 Conn_Coaxial, J102 Conn_Coaxial, J103 Conn_Coaxial, J104 Conn_Coaxial, J105 Conn_02x14_Odd_Even

Commit message: Added pull resistors to deselect and powerdown by defalut all ICs and more GND vias!
Signed-off-by: Alexis Jeandet <alexis.jeandet@member.fsf.org>
Parts:
- added R101, R102: 100k, Resistor_SMD:R_0603_1608Metric_Pad1.05x0.95mm_HandSolder, symbol Device:R
Connections:
- net DVDD: now also R102.1
- net GND: now also R101.2
- net ~CS: now also R102.2
- net ~POWERDOWN: now also R101.1
Changed lines of the file:
@@
 	1    0    0    -1
 $EndComp
+$Comp
+L Device:R R101
+U 1 1 5F05FD5F
+P 9025 1925
+F 0 "R101" H 9095 1971 50  0000 L CNN
+F 1 "100k" H 9095 1880 50  0000 L CNN
+F 2 "Resistor_SMD:R_0603_1608Metric_Pad1.05x0.95mm_HandSolder" V 8955 1925 50  0001 C CNN
+F 3 "~" H 9025 1925 50  0001 C CNN
+	1    9025 1925
+	1    0    0    -1
+$EndComp
+Text Label 9150 1650 0    50   ~ 0
+~POWERDOWN
+$Comp
+L power:GND #PWR0115
+U 1 1 5F06182F
+P 9025 2175
+F 0 "#PWR0115" H 9025 1925 50  0001 C CNN
+F 1 "GND" H 9175 2125 50  0000 C CNN
+F 2 "" H 9025 2175 50  0001 C CNN
+F 3 "" H 9025 2175 50  0001 C CNN
+	1    9025 2175
+	1    0    0    -1
+$EndComp
+Wire Wire Line
+	9025 2175 9025 2075
+Wire Wire Line
+	9025 1775 9025 1650
+Wire Wire Line
+	9025 1650 9150 1650
+$Comp
+L Device:R R102
+U 1 1 5F0645C0
+P 9800 1300
+F 0 "R102" H 9870 1346 50  0000 L CNN
+F 1 "100k" H 9870 1255 50  0000 L CNN
+F 2 "Resistor_SMD:R_0603_1608Metric_Pad1.05x0.95mm_HandSolder" V 9730 1300 50  0001 C CNN
+F 3 "~" H 9800 1300 50  0001 C CNN
+	1    9800 1300
+	1    0    0    -1
+$EndComp
+Text Label 9950 1650 0    50   ~ 0
+~CS
+Wire Wire Line
+	9800 1450 9800 1650
+Wire Wire Line
+	9800 1650 9950 1650
+Text Label 10000 1025 0    50   ~ 0
+DVDD
+Wire Wire Line
+	10000 1025 9800 1025
+Wire Wire Line
+	9800 1025 9800 1150
 $EndSCHEMATC
