File: STM32Scope.kicad_pcb (KiCad board)
At the start: 4 copper layers, 50.8 x 40.6 mm, 43 parts, among them J101 Conn_Coaxial, J102 Conn_Coaxial, J103 Conn_Coaxial, J104 Conn_Coaxial, J105 Conn_02x14_Odd_Even, U303 ADS92x4R, U401 THS4551, U501 THS4551

Commit message: Added pull resistors to deselect and powerdown by defalut all ICs and more GND vias!
Signed-off-by: Alexis Jeandet <alexis.jeandet@member.fsf.org>
Parts:
- added R101: 100k, Resistor_SMD:R_0603_1608Metric_Pad1.05x0.95mm_HandSolder, F.Cu at (95.5, 94.5)
- added R102: 100k, Resistor_SMD:R_0603_1608Metric_Pad1.05x0.95mm_HandSolder, B.Cu at (88.4, 104.6)
Routing:
- net /DVDD: track 22.3 -> 26.1 mm
- net /~CS: track 13.7 -> 16.9 mm
- net /~POWERDOWN: track 75.9 -> 79.0 mm
- net GND: vias 228 -> 252

Commit message: Few cleanups
Signed-off-by: Alexis Jeandet <alexis.jeandet@member.fsf.org>
Parts:
- moved C304 0.92 mm to (85.3, 100.6)
- moved C302 0.76 mm to (87.4, 98.1)
- moved C303 0.71 mm to (86.4, 109.1)
Routing:
- net /DVDD: track 26.1 -> 24.0 mm
- net /AVDD: track 76.1 -> 74.0 mm
- net GND: vias 252 -> 257

Commit message: Ready for manufacturing v1.0
Signed-off-by: Alexis Jeandet <alexis.jeandet@member.fsf.org>
Parts:
- moved C304 1.44 mm to (86.4, 99.6), turned to 270 degrees
Routing:
- net /~POWERDOWN: track 79.0 -> 78.5 mm
- net GND: vias 257 -> 296
- added copper zone on F.Cu, net Net-(C305-Pad2)
- added copper zone on F.Cu, net Net-(C306-Pad1)
Other:
- board text added: "STM32Scope 1.0"
